File: SampleTags.kicad_pcb (KiCad board)
At the start: 2 copper layers, 47.5 x 47.7 mm, 7 parts

Commit message: Update SampleTags.kicad_pcb
Parts:
- removed G***: LOGO, BadgePiratesLogo:BadgePiratesURL_B.SLK
- removed G***: BP Logo, BadgePiratesLogo:BPSkull_Distressed_B.SILK
- removed G***: BP LOGO, BadgePiratesLogo:BPSkull_Distressed_F.CU
- removed REF**: 3.5mm_lapel_pin, BadgePirates:Hole_3mm_lapel_pin
- removed REF**: 12x5 SLOT, BadgePirates:Slot_12x5mm
- removed REF**: 5.5mm, BadgePirates:Hole_5.5mm
- removed kibuzzard-63169E39: G***, kibuzzard-63169E39
- added G***10: BP Logo, BadgePiratesLogo:BPSkull_Distressed_B.SILK, F.Cu at (104.3, 178.2)
- added G***11: LOGO, BadgePiratesLogo:BadgePiratesURL_B.SLK, F.Cu at (100.8, 160.6)
- added G***12: BP LOGO, BadgePiratesLogo:BPSkull_Distressed_F.CU, B.Cu at (121.0, 148.2)
- added G***13: BP Logo, BadgePiratesLogo:BPSkull_Distressed_B.SILK, F.Cu at (153.4, 178.2)
- added G***14: LOGO, BadgePiratesLogo:BadgePiratesURL_B.SLK, F.Cu at (149.9, 160.6)
- added G***15: BP LOGO, BadgePiratesLogo:BPSkull_Distressed_F.CU, B.Cu at (170.1, 148.2)
- added G***4: BP Logo, BadgePiratesLogo:BPSkull_Distressed_B.SILK, F.Cu at (104.3, 129.1)
- added G***5: LOGO, BadgePiratesLogo:BadgePiratesURL_B.SLK, F.Cu at (100.8, 111.5)
- added G***6: BP LOGO, BadgePiratesLogo:BPSkull_Distressed_F.CU, B.Cu at (121.0, 99.1)
- added G***7: BP Logo, BadgePiratesLogo:BPSkull_Distressed_B.SILK, F.Cu at (153.4, 129.1)
- added G***8: LOGO, BadgePiratesLogo:BadgePiratesURL_B.SLK, F.Cu at (149.9, 111.5)
- added G***9: BP LOGO, BadgePiratesLogo:BPSkull_Distressed_F.CU, B.Cu at (170.1, 99.1)
- added REF**10: 3.5mm_lapel_pin, BadgePirates:Hole_3mm_lapel_pin, F.Cu at (140.5, 185.3)
- added REF**11: 5.5mm, BadgePirates:Hole_5.5mm, F.Cu at (139.5, 145.6)
- added REF**12: 12x5 SLOT, BadgePirates:Slot_12x5mm, F.Cu at (104.4, 145.5)
- added REF**13: 3.5mm_lapel_pin, BadgePirates:Hole_3mm_lapel_pin, F.Cu at (189.6, 185.3)
- added REF**14: 5.5mm, BadgePirates:Hole_5.5mm, F.Cu at (188.6, 145.6)
- added REF**15: 12x5 SLOT, BadgePirates:Slot_12x5mm, F.Cu at (153.5, 145.5)
- added REF**4: 3.5mm_lapel_pin, BadgePirates:Hole_3mm_lapel_pin, F.Cu at (140.5, 136.2)
- added REF**5: 5.5mm, BadgePirates:Hole_5.5mm, F.Cu at (139.5, 96.5)
- added REF**6: 12x5 SLOT, BadgePirates:Slot_12x5mm, F.Cu at (104.4, 96.4)
- added REF**7: 3.5mm_lapel_pin, BadgePirates:Hole_3mm_lapel_pin, F.Cu at (189.6, 136.2)
- added REF**8: 5.5mm, BadgePirates:Hole_5.5mm, F.Cu at (188.6, 96.5)
- added REF**9: 12x5 SLOT, BadgePirates:Slot_12x5mm, F.Cu at (153.5, 96.4)
- added kibuzzard-63169E1: G***, kibuzzard-63169E39, B.Cu at (152.6, 137.8)
- added kibuzzard-63169E2: G***, kibuzzard-63169E39, B.Cu at (103.5, 137.8)
- added kibuzzard-63169E3: G***, kibuzzard-63169E39, B.Cu at (103.5, 186.9)
- added kibuzzard-63169E4: G***, kibuzzard-63169E39, B.Cu at (152.6, 186.9)
Routing:
- net (no net): vias 2 -> 8
Other:
- board size 47.5 x 47.7 mm -> 96.6 x 96.8 mm
